File: BPS-ShuntResistorPCB.sch (KiCad schematic (older format))
At the start: 3 parts, among them J1 Amp_Conn

Commit message: Initial board dev (#2)
* added logos and conn footprint

* updated connector to match ampere board

* added resistor footprint

* needs to be reviewed

* implemented edits

* fixed typo

* more edits

* more edits

* Creates gerbers

* Creates gerber edits to the PCB

* Creates gerbers

Co-authored-by: Elijah Gonzalez <elijah.gonzalez.utexasedu>
Co-authored-by: Hannah Lee <hannahslee@utexas.edu>
Parts:
- removed J1: Amp_Conn, symbol Connector_Generic:Conn_01x04
- added H1, H2: MountingHole, MountingHole:MountingHole_2.7mm_M2.5, symbol Mechanical:MountingHole
- added J1: Amp_Conn, UTSVT_Connectors:Power_Metal_Strip_Battery_Shunt_Resistor_4_Pin_Connector, symbol Connector_Generic:Conn_02x02_Counter_Clockwise
- added LOGO1: UTSVT, UTSVT_Special:UTSVT_Logo_Symbol, symbol utsvt-misc:Logo_Placeholder
- added LOGO2: Dr Hallock, UTSVT_Special:Hallock_Image_Tiny, symbol utsvt-misc:Logo_Placeholder
- R1: footprint Resistor_SMD:R_0805_2012Metric -> UTSVT_Passive:Power_Metal_Strip_Battery_Shunt_Resistor
Connections:
- net ETS: now also TH1.2, J1.1 (Pin_1); no longer TH1.1
- net GND: now also TH1.1, J1.4 (Pin_4); no longer TH1.2
- net RSHH: now also J1.3 (Pin_3)
- net RSHL: now also J1.2 (Pin_2)
Other:
- moved on the sheet: R1, TH1
Changed lines of the file:
@@
 Comment4 ""
 $EndDescr
-Wire Wire Line
-	6650 4250 6650 4000
-Wire Wire Line
-	6650 4000 5950 4000
-Wire Wire Line
-	5950 4300 5950 4350
-Wire Wire Line
-	5950 4350 6650 4350
-Wire Wire Line
-	6650 4550 6650 4850
-Wire Wire Line
-	6650 4850 5950 4850
-Wire Wire Line
-	5950 4450 6650 4450
-Text Label 6450 4000 0    50   ~ 0
+Text Label 5750 4750 1    50   ~ 0
 RSHH
-Text Label 6450 4350 0    50   ~ 0
+Text Label 5250 4550 3    50   ~ 0
 RSHL
-Text Label 6450 4450 0    50   ~ 0
+Text Label 5250 3950 1    50   ~ 0
 ETS
-Text Label 6450 4850 0    50   ~ 0
+Text Label 5750 3950 1    50   ~ 0
 GND
 $Comp
-L Connector_Generic:Conn_01x04 J1
-U 1 1 5F54708B
-P 6850 4350
-F 0 "J1" H 6950 4400 50  0000 L CNN
-F 1 "Amp_Conn" H 6950 4300 50  0000 L CNN
-F 2 "" H 6850 4350 50  0001 C CNN
-F 3 "~" H 6850 4350 50  0001 C CNN
-	1    6850 4350
+L Device:Thermistor TH1
+U 1 1 5F548CAA
+P 5500 3550
+F 0 "TH1" H 5605 3596 50  0000 L CNN
+F 1 "100" H 5605 3505 50  0000 L CNN
+F 2 "Resistor_SMD:R_0805_2012Metric" H 5500 3550 50  0001 C CNN
+F 3 "~" H 5500 3550 50  0001 C CNN
+	1    5500 3550
+	0    1    1    0
+$EndComp
+$Comp
+L utsvt-misc:Logo_Placeholder LOGO1
+U 1 1 5F53FE42
+P 6250 4500
+F 0 "LOGO1" H 6250 4650 50  0001 C CNN
+F 1 "UTSVT" H 6390 4500 50  0000 L CNN
+F 2 "UTSVT_Special:UTSVT_Logo_Symbol" H 6250 4575 50  0001 C CNN
+F 3 "" H 6250 4575 50  0001 C CNN
+	1    6250 4500
+	1    0    0    -1
+$EndComp
+$Comp
+L utsvt-misc:Logo_Placeholder LOGO2
+U 1 1 5F5407D9
+P 6250 4750
+F 0 "LOGO2" H 6250 4900 50  0001 C CNN
+F 1 "Dr Hallock" H 6390 4750 50  0000 L CNN
+F 2 "UTSVT_Special:Hallock_Image_Tiny" H 6250 4825 50  0001 C CNN
+F 3 "" H 6250 4825 50  0001 C CNN
+	1    6250 4750
 	1    0    0    -1
 $EndComp
@@
 L Device:R R1
 U 1 1 5F548200
-P 5950 4150
-F 0 "R1" H 6020 4196 50  0000 L CNN
-F 1 "100u" H 6020 4105 50  0000 L CNN
-F 2 "Resistor_SMD:R_0805_2012Metric" V 5880 4150 50  0001 C CNN
-F 3 "~" H 5950 4150 50  0001 C CNN
-	1    5950 4150
+P 5500 4850
+F 0 "R1" H 5570 4896 50  0000 L CNN
+F 1 "100u" H 5570 4805 50  0000 L CNN
+F 2 "UTSVT_Passive:Power_Metal_Strip_Battery_Shunt_Resistor" V 5430 4850 50  0001 C CNN
+F 3 "~" H 5500 4850 50  0001 C CNN
+	1    5500 4850
+	0    1    1    0
+$EndComp
+$Comp
+L Connector_Generic:Conn_02x02_Counter_Clockwise J1
+U 1 1 5F55AEC1
+P 5450 4350
+F 0 "J1" H 5500 4567 50  0000 C CNN
+F 1 "Amp_Conn" H 5500 4476 50  0000 C CNN
+F 2 "UTSVT_Connectors:Power_Metal_Strip_Battery_Shunt_Resistor_4_Pin_Connector" H 5450 4350 50  0001 C CNN
+F 3 "~" H 5450 4350 50  0001 C CNN
+	1    5450 4350
+	1    0    0    -1
+$EndComp
+Wire Wire Line
+	5250 4350 5250 3550
+Wire Wire Line
+	5250 3550 5300 3550
+Wire Wire Line
+	5750 4350 5750 3550
+Wire Wire Line
+	5750 3550 5700 3550
+Wire Wire Line
+	5250 4450 5250 4850
+Wire Wire Line
+	5250 4850 5350 4850
+Wire Wire Line
+	5650 4850 5750 4850
+Wire Wire Line
+	5750 4850 5750 4450
+$Comp
+L Mechanical:MountingHole H1
+U 1 1 5F6F5E19
+P 3000 2100
+F 0 "H1" H 3100 2146 50  0000 L CNN
+F 1 "MountingHole" H 3100 2055 50  0000 L CNN
+F 2 "MountingHole:MountingHole_2.7mm_M2.5" H 3000 2100 50  0001 C CNN
+F 3 "~" H 3000 2100 50  0001 C CNN
+	1    3000 2100
 	1    0    0    -1
 $EndComp
 $Comp
-L Device:Thermistor TH1
-U 1 1 5F548CAA
-P 5950 4650
-F 0 "TH1" H 6055 4696 50  0000 L CNN
-F 1 "100" H 6055 4605 50  0000 L CNN
-F 2 "Resistor_SMD:R_0805_2012Metric" H 5950 4650 50  0001 C CNN
-F 3 "~" H 5950 4650 50  0001 C CNN
-	1    5950 4650
+L Mechanical:MountingHole H2
+U 1 1 5F6F8A03
+P 2950 2900
+F 0 "H2" H 3050 2946 50  0000 L CNN
+F 1 "MountingHole" H 3050 2855 50  0000 L CNN
+F 2 "MountingHole:MountingHole_2.7mm_M2.5" H 2950 2900 50  0001 C CNN
+F 3 "~" H 2950 2900 50  0001 C CNN
+	1    2950 2900
 	1    0    0    -1
 $EndComp
